Commit message: Fixed friction in simulation and tunned PID in Gazebo

File: first_description/robot/first.gazebo.xacro (robot description, xacro)
@@ -8,5 +8,7 @@
     </plugin>
   </gazebo>
- <gazebo reference="base_link">
+  <gazebo reference="base_link">
+    <mu1>0.2</mu1>
+    <mu2>0.2</mu2>
     <material>Gazebo/White</material>
   </gazebo>

File: first_description/robot/robot.urdf.xacro (robot description, xacro)
@@ -19,5 +19,5 @@
     </visual>
     <xacro:box_collision width="${base_width}" depth="${base_height}" height="${base_length}"/>
-    <xacro:box_inertia mass="0.2" width="${base_width}" depth="${base_height}" height="${base_length}"/>
+    <xacro:box_inertia mass="100.2" width="${base_width}" depth="${base_height}" height="${base_length}"/>
   </link>
   <link name="wheel_holder">
@@ -51,5 +51,5 @@
     <axis xyz="0 0 1" />
     <limit effort="100" velocity="100" />
-    <dynamics damping="0.01" friction="100.0" />
+    <dynamics damping="0.01" friction="0.0" />
   </joint>
   <transmission name="wheel_transmission">
